File: kicad/TL072.kicad_sch (KiCad schematic)
At the start: 22 parts, among them J2 AudioJack3_SwitchTR, J5 x out, J6 y out, U1 TL072, U2 X galvo, U3 Y TL072

Commit message: Update KiCad source files
Parts:
- R1, R10, R11, R12, R13, R14, R2, R3, R4, R5, R6, R7, R8, R9: footprint Resistor_SMD:R_0603_1608Metric -> Resistor_SMD:R_0805_2012Metric_Pad1.20x1.40mm_HandSolder
Changed lines of the file:
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@@
 			)
 		)
-		(property "Footprint" "Resistor_SMD:R_0603_1608Metric"
+		(property "Footprint" "Resistor_SMD:R_0805_2012Metric_Pad1.20x1.40mm_HandSolder"
 			(at 204.47 94.742 90)
 			(effects
@@
 		)
 		(instances
-			(project "teensy 4.1 laser"
+			(project "teensy-4-galvos"
 				(path "/a482f7a8-c6b1-4177-8f46-04920beda042/6d17ce7a-96b0-4268-8807-23a23df5693a"
 					(reference "R13")
@@
 		)
 		(instances
-			(project "teensy 4.1 laser"
+			(project "teensy-4-galvos"
 				(path "/a482f7a8-c6b1-4177-8f46-04920beda042/6d17ce7a-96b0-4268-8807-23a23df5693a"
 					(reference "#PWR010")
@@
 		)
 		(instances
-			(project "teensy 4.1 laser"
+			(project "teensy-4-galvos"
 				(path "/a482f7a8-c6b1-4177-8f46-04920beda042/6d17ce7a-96b0-4268-8807-23a23df5693a"
 					(reference "U3")
@@
 		)
 		(instances
-			(project "teensy 4.1 laser"
+			(project "teensy-4-galvos"
 				(path "/a482f7a8-c6b1-4177-8f46-04920beda042/6d17ce7a-96b0-4268-8807-23a23df5693a"
 					(reference "J5")
@@
 		)
 		(instances
-			(project "teensy 4.1 laser"
+			(project "teensy-4-galvos"
 				(path "/a482f7a8-c6b1-4177-8f46-04920beda042/6d17ce7a-96b0-4268-8807-23a23df5693a"
 					(reference "#PWR07")
@@
 		)
 		(instances
-			(project "teensy 4.1 laser"
+			(project "teensy-4-galvos"
 				(path "/a482f7a8-c6b1-4177-8f46-04920beda042/6d17ce7a-96b0-4268-8807-23a23df5693a"
 					(reference "U2")
@@
 			)
 		)
-		(property "Footprint" "Resistor_SMD:R_0603_1608Metric"
+		(property "Footprint" "Resistor_SMD:R_0805_2012Metric_Pad1.20x1.40mm_HandSolder"
 			(at 158.75 116.332 90)
 			(effects
@@
 		)
 		(instances
-			(project "teensy 4.1 laser"
+			(project "teensy-4-galvos"
 				(path "/a482f7a8-c6b1-4177-8f46-04920beda042/6d17ce7a-96b0-4268-8807-23a23df5693a"
 					(reference "R8")
@@
 			)
 		)
-		(property "Footprint" "Resistor_SMD:R_0603_1608Metric"
+		(property "Footprint" "Resistor_SMD:R_0805_2012Metric_Pad1.20x1.40mm_HandSolder"
 			(at 158.75 71.882 90)
 			(effects
@@
 		)
 		(instances
-			(project "teensy 4.1 laser"
+			(project "teensy-4-galvos"
 				(path "/a482f7a8-c6b1-4177-8f46-04920beda042/6d17ce7a-96b0-4268-8807-23a23df5693a"
 					(reference "R6")
@@
 		)
 		(instances
-			(project "teensy 4.1 laser"
+			(project "teensy-4-galvos"
 				(path "/a482f7a8-c6b1-4177-8f46-04920beda042/6d17ce7a-96b0-4268-8807-23a23df5693a"
 					(reference "U1")
@@
 			)
 		)
-		(property "Footprint" "Resistor_SMD:R_0603_1608Metric"
+		(property "Footprint" "Resistor_SMD:R_0805_2012Metric_Pad1.20x1.40mm_HandSolder"
 			(at 104.648 118.11 90)
 			(effects
@@
 		)
 		(instances
-			(project "teensy 4.1 laser"
+			(project "teensy-4-galvos"
 				(path "/a482f7a8-c6b1-4177-8f46-04920beda042/6d17ce7a-96b0-4268-8807-23a23df5693a"
 					(reference "R2")
@@
 		)
 		(instances
-			(project "teensy 4.1 laser"
+			(project "teensy-4-galvos"
 				(path "/a482f7a8-c6b1-4177-8f46-04920beda042/6d17ce7a-96b0-4268-8807-23a23df5693a"
 					(reference "#FLG03")
@@
 			)
 		)
-		(property "Footprint" "Resistor_SMD:R_0603_1608Metric"
+		(property "Footprint" "Resistor_SMD:R_0805_2012Metric_Pad1.20x1.40mm_HandSolder"
 			(at 177.8 79.502 90)
 			(effects
@@
 		)
 		(instances
-			(project "teensy 4.1 laser"
+			(project "teensy-4-galvos"
 				(path "/a482f7a8-c6b1-4177-8f46-04920beda042/6d17ce7a-96b0-4268-8807-23a23df5693a"
 					(reference "R9")
@@
 			)
 		)
-		(property "Footprint" "Resistor_SMD:R_0603_1608Metric"
+		(property "Footprint" "Resistor_SMD:R_0805_2012Metric_Pad1.20x1.40mm_HandSolder"
 			(at 177.8 123.952 90)
 			(effects
@@
 		)
 		(instances
-			(project "teensy 4.1 laser"
+			(project "teensy-4-galvos"
 				(path "/a482f7a8-c6b1-4177-8f46-04920beda042/6d17ce7a-96b0-4268-8807-23a23df5693a"
 					(reference "R10")
@@
 		)
 		(instances
-			(project "teensy 4.1 laser"
+			(project "teensy-4-galvos"
 				(path "/a482f7a8-c6b1-4177-8f46-04920beda042/6d17ce7a-96b0-4268-8807-23a23df5693a"
 					(reference "J2")
@@
 			)
 		)
-		(property "Footprint" "Resistor_SMD:R_0603_1608Metric"
+		(property "Footprint" "Resistor_SMD:R_0805_2012Metric_Pad1.20x1.40mm_HandSolder"
 			(at 204.47 69.342 90)
 			(effects
@@
 		)
 		(instances
-			(project "teensy 4.1 laser"
+			(project "teensy-4-galvos"
 				(path "/a482f7a8-c6b1-4177-8f46-04920beda042/6d17ce7a-96b0-4268-8807-23a23df5693a"
 					(reference "R12")
@@
 			)
 		)
-		(property "Footprint" "Resistor_SMD:R_0603_1608Metric"
+		(property "Footprint" "Resistor_SMD:R_0805_2012Metric_Pad1.20x1.40mm_HandSolder"
 			(at 129.54 70.612 90)
 			(effects
@@
 		)
 		(instances
-			(project "teensy 4.1 laser"
+			(project "teensy-4-galvos"
 				(path "/a482f7a8-c6b1-4177-8f46-04920beda042/6d17ce7a-96b0-4268-8807-23a23df5693a"
 					(reference "R3")
@@
 			)
 		)
-		(property "Footprint" "Resistor_SMD:R_0603_1608Metric"
+		(property "Footprint" "Resistor_SMD:R_0805_2012Metric_Pad1.20x1.40mm_HandSolder"
 			(at 204.47 113.792 90)
 			(effects
@@
 		)
 		(instances
-			(project "teensy 4.1 laser"
+			(project "teensy-4-galvos"
 				(path "/a482f7a8-c6b1-4177-8f46-04920beda042/6d17ce7a-96b0-4268-8807-23a23df5693a"
 					(reference "R14")
@@
 		)
 		(instances
-			(project "teensy 4.1 laser"
+			(project "teensy-4-galvos"
 				(path "/a482f7a8-c6b1-4177-8f46-04920beda042/6d17ce7a-96b0-4268-8807-23a23df5693a"
 					(reference "#PWR06")
@@
 			)
 		)
-		(property "Footprint" "Resistor_SMD:R_0603_1608Metric"
+		(property "Footprint" "Resistor_SMD:R_0805_2012Metric_Pad1.20x1.40mm_HandSolder"
 			(at 158.75 92.202 90)
 			(effects
@@
 		)
 		(instances
-			(project "teensy 4.1 laser"
+			(project "teensy-4-galvos"
 				(path "/a482f7a8-c6b1-4177-8f46-04920beda042/6d17ce7a-96b0-4268-8807-23a23df5693a"
 					(reference "R7")
@@
 		)
 		(instances
-			(project "teensy 4.1 laser"
+			(project "teensy-4-galvos"
 				(path "/a482f7a8-c6b1-4177-8f46-04920beda042/6d17ce7a-96b0-4268-8807-23a23df5693a"
 					(reference "#PWR011")
@@
 		)
 		(instances
-			(project "teensy 4.1 laser"
+			(project "teensy-4-galvos"
 				(path "/a482f7a8-c6b1-4177-8f46-04920beda042/6d17ce7a-96b0-4268-8807-23a23df5693a"
 					(reference "J6")
@@
 		)
 		(instances
-			(project "teensy 4.1 laser"
+			(project "teensy-4-galvos"
 				(path "/a482f7a8-c6b1-4177-8f46-04920beda042/6d17ce7a-96b0-4268-8807-23a23df5693a"
 					(reference "#PWR08")
@@
 		)
 		(instances
-			(project "teensy 4.1 laser"
+			(project "teensy-4-galvos"
 				(path "/a482f7a8-c6b1-4177-8f46-04920beda042/6d17ce7a-96b0-4268-8807-23a23df5693a"
 					(reference "U1")
@@
 		)
 		(instances
-			(project "teensy 4.1 laser"
+			(project "teensy-4-galvos"
 				(path "/a482f7a8-c6b1-4177-8f46-04920beda042/6d17ce7a-96b0-4268-8807-23a23df5693a"
 					(reference "U3")
@@
 			)
 		)
-		(property "Footprint" "Resistor_SMD:R_0603_1608Metric"
+		(property "Footprint" "Resistor_SMD:R_0805_2012Metric_Pad1.20x1.40mm_HandSolder"
 			(at 204.47 50.292 90)
 			(effects
@@
 		)
 		(instances
-			(project "teensy 4.1 laser"
+			(project "teensy-4-galvos"
 				(path "/a482f7a8-c6b1-4177-8f46-04920beda042/6d17ce7a-96b0-4268-8807-23a23df5693a"
 					(reference "R11")
@@
 			)
 		)
-		(property "Footprint" "Resistor_SMD:R_0603_1608Metric"
+		(property "Footprint" "Resistor_SMD:R_0805_2012Metric_Pad1.20x1.40mm_HandSolder"
 			(at 104.648 72.39 90)
 			(effects
@@
 		)
 		(instances
-			(project "teensy 4.1 laser"
+			(project "teensy-4-galvos"
 				(path "/a482f7a8-c6b1-4177-8f46-04920beda042/6d17ce7a-96b0-4268-8807-23a23df5693a"
 					(reference "R1")
@@
 		)
 		(instances
-			(project "teensy 4.1 laser"
+			(project "teensy-4-galvos"
 				(path "/a482f7a8-c6b1-4177-8f46-04920beda042/6d17ce7a-96b0-4268-8807-23a23df5693a"
 					(reference "RV1")
@@
 			)
 		)
-		(property "Footprint" "Resistor_SMD:R_0603_1608Metric"
+		(property "Footprint" "Resistor_SMD:R_0805_2012Metric_Pad1.20x1.40mm_HandSolder"
 			(at 158.75 47.752 90)
 			(effects
@@
 		)
 		(instances
-			(project "teensy 4.1 laser"
+			(project "teensy-4-galvos"
 				(path "/a482f7a8-c6b1-4177-8f46-04920beda042/6d17ce7a-96b0-4268-8807-23a23df5693a"
 					(reference "R5")
@@
 			)
 		)
-		(property "Footprint" "Resistor_SMD:R_0603_1608Metric"
+		(property "Footprint" "Resistor_SMD:R_0805_2012Metric_Pad1.20x1.40mm_HandSolder"
 			(at 129.54 116.332 90)
 			(effects
@@
 		)
 		(instances
-			(project "teensy 4.1 laser"
+			(project "teensy-4-galvos"
 				(path "/a482f7a8-c6b1-4177-8f46-04920beda042/6d17ce7a-96b0-4268-8807-23a23df5693a"
 					(reference "R4")
@@
 		)
 		(instances
-			(project "teensy 4.1 laser"
+			(project "teensy-4-galvos"
 				(path "/a482f7a8-c6b1-4177-8f46-04920beda042/6d17ce7a-96b0-4268-8807-23a23df5693a"
 					(reference "#PWR09")
@@
 		)
 		(instances
-			(project "teensy 4.1 laser"
+			(project "teensy-4-galvos"
 				(path "/a482f7a8-c6b1-4177-8f46-04920beda042/6d17ce7a-96b0-4268-8807-23a23df5693a"
 					(reference "RV2")
@@
 		)
 		(instances
-			(project "teensy 4.1 laser"
+			(project "teensy-4-galvos"
 				(path "/a482f7a8-c6b1-4177-8f46-04920beda042/6d17ce7a-96b0-4268-8807-23a23df5693a"
 					(reference "U2")

Commit message: Update KiCad board files
Parts:
- removed J5: x out, Connector_Molex:Molex_KK-254_AE-6410-03A_1x03_P2.54mm_Vertical, symbol Connector:Screw_Terminal_01x03
- removed J6: y out, Connector_Molex:Molex_KK-254_AE-6410-03A_1x03_P2.54mm_Vertical, symbol Connector:Screw_Terminal_01x03
- added J3: (no value), Connector_JST:JST_XH_B3B-XH-A_1x03_P2.50mm_Vertical, symbol Connector:Screw_Terminal_01x03
- R1, R10, R11, R12, R13, R14, R2, R3, R4, R5, R6, R7, R8, R9: footprint Resistor_SMD:R_0805_2012Metric_Pad1.20x1.40mm_HandSolder -> Resistor_SMD:R_0603_1608Metric
- RV1, RV2: footprint Potentiometer_THT:Potentiometer_Bourns_3296X_Horizontal -> Potentiometer_THT:Potentiometer_Bourns_3386P_Vertical
Connections:
- net Ax_Sleeve_OUT is gone; now on net GND: J2.S
- net GND: now also J3.3 (Pin_3)
- net at R12.1: now also J3.1 (Pin_1)
- net at R14.1: now also J3.2 (Pin_2)
- no-connect marks 5 -> 6
