File: kicad/teensy-4-galvos.kicad_pcb (KiCad board)
At the start: 2 copper layers, 70 x 40 mm, 32 parts, among them J1 +15 G -15, J2 AudioJack3_SwitchTR, J3 +15 G -15, J7 405nm, U1 TL072, U2 X galvo, U3 Y TL072, U4 Teensy4.0

Commit message: Preserve reviewed local project changes before cleanup [skip ci]
Routing:
- net GND: track 122.5 -> 0.00 mm
- net -15V: track 94.3 -> 0.00 mm, vias 1 -> 0
- net Net-(R4-Pad1): track 47.8 -> 0.00 mm, vias 2 -> 0
- net +15V: track 43.4 -> 0.00 mm
- net Net-(R3-Pad1): track 36.2 -> 0.00 mm
- net Net-(J3-Pin_2): track 35.2 -> 0.00 mm, vias 1 -> 0
- net /laser en: track 34.7 -> 0.00 mm
- net Net-(U1B--): track 33.2 -> 0.00 mm, vias 1 -> 0
- net Net-(U1A--): track 32.1 -> 0.00 mm, vias 1 -> 0
- net Net-(J3-Pin_1): track 29.3 -> 0.00 mm
- net Net-(R4-Pad2): track 29.2 -> 0.00 mm, vias 1 -> 0
- net Ax_Ring_OUT: track 29.1 -> 0.00 mm
- net Net-(R12-Pad2): track 13.3 -> 0.00 mm
- net Net-(U2B--): track 13.2 -> 0.00 mm
- net Net-(R10-Pad1): track 10.4 -> 0.00 mm
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- removed copper zone on B.Cu, net GND
Other:
- outline, holes or cut-outs redrawn
