File: kicad/teensy-4-galvos.kicad_sch (KiCad schematic)
At the start: 12 parts, among them J1 +15 G -15, J7 405nm, U1 TL072, U2 X galvo, U3 Y TL072, U4 Teensy4.0, U5 LM2596S-5

Commit message: Update KiCad source files
Parts:
- removed C1: 100µF, Capacitor_SMD:C_1206_3216Metric, symbol Device:C
- removed C2: 220µF, Capacitor_SMD:C_1206_3216Metric, symbol Device:C
- removed C3: 0.1µF, Capacitor_SMD:C_0603_1608Metric, symbol Device:C_Small
- removed D1: 1N5824, Diode_SMD:D_SMA, symbol Device:D_Schottky
- removed L1: 68µH, Inductor_SMD:L_Bourns-SRN6028, symbol Device:L
- removed U5: LM2596S-5, Package_TO_SOT_SMD:TO-252-5_TabPin3, symbol Regulator_Switching:LM2596S-5
Other:
- note removed: "5V regulator"

Commit message: Update KiCad board files
Parts:
- added C1, C2, C3, C4, C5, C6: 0.1uF, Capacitor_SMD:C_0603_1608Metric_Pad1.08x0.95mm_HandSolder, symbol Device:C_Small
- added C7, C8: 10uF, Capacitor_SMD:C_0805_2012Metric_Pad1.18x1.45mm_HandSolder, symbol Device:C_Small
- J1: footprint Connector_Molex:Molex_KK-254_AE-6410-03A_1x03_P2.54mm_Vertical -> Connector_JST:JST_XH_B3B-XH-A_1x03_P2.50mm_Vertical
Connections:
- net +15V: now also C4.1, C5.1, C6.1, C8.1
- net -15V: now also C1.1, C2.1, C3.1, C7.1
- net GND: now also C1.2, C2.2, C3.2, C4.2, C5.2, C6.2, C7.2, C8.2; no longer U4.1 (GND)
- no-connect marks 50 -> 51
